Commit message: add tool and positioner frames to urdf

File: urdf/positioner.xacro (robot description, xacro)
@@ -10,5 +10,5 @@
     <axis xyz="0 0 1"/>
     <parent link="world"/>
-    <child link="$(arg prefix)rotary_table_link"/>
+    <child link="$(arg prefix)rotary_table_base"/>
   </joint>
 </robot>

File: urdf/positioner_macro.xacro (robot description, xacro)
@@ -17,10 +17,11 @@
       </collision>
     </link>
-    <link name="${prefix}positioner_link">
+    <link name="${prefix}rotary_table_top"/>
+    <link name="${prefix}positioner_base">
         <visual>
         <geometry>
           <mesh filename="package://hydra_description/meshes/hydra_positioner.dae"/>
         </geometry>
-        <origin rpy="0.0 0.0 0.0" xyz="0 0 0.1778"/>
+        <origin rpy="0.0 0.0 0.0" xyz="0 0 0"/>
       </visual>
       <collision>
@@ -31,10 +32,23 @@
       </collision>
     </link>
+    <link name="${prefix}positioner"/>
     <!-- joint list -->
-    <joint name="${prefix}positioner_joint" type="continuous">
+    <joint name="{prefix}rotary_table_top_base" type="fixed">
+      <parent link="${prefix}rotary_table_base"/>
+      <child link="${prefix}rotary_table_top"/>
+      <axis xyz="0 0 0"/>
+      <origin rpy="0.0 0.0 0.0" xyz="0 0 0.1778"/>
+    </joint>
+    <joint name="${prefix}rotary_table_positioner" type="continuous">
       <origin rpy="0.0 0.0 0.0" xyz="0 0 0"/>
       <axis xyz="0 0 1"/>
-      <parent link="${prefix}rotary_table_base"/>
-      <child link="${prefix}positioner_link"/>
+      <parent link="${prefix}rotary_table_top"/>
+      <child link="${prefix}positioner_base"/>
+    </joint>
+    <joint name="${prefix}positioner_joint" type="fixed">
+      <origin rpy="0.0 0.0 0.0" xyz="0 0 0.03175"/>
+      <axis xyz="0 0 1"/>
+      <parent link="${prefix}positioner_base"/>
+      <child link="${prefix}positioner"/>
     </joint>
   </xacro:macro>

File: urdf/za_typhoon_macro.xacro (robot description, xacro)
@@ -5,5 +5,5 @@
     <xacro:za_macro prefix="${prefix}" tool0_trans="${tool0_trans}" tool0_rot="${tool0_trans}" tool0_fixed="True"/>
     <!-- link list -->
-    <link name="${prefix}typhoon_extruder">
+    <link name="${prefix}typhoon_extruder_base">
         <visual>
         <geometry>
@@ -19,11 +19,20 @@
       </collision>
     </link>
-    <!-- attach extruder to link_6 -->
+    <link name="${prefix}typhoon_extruder">
+      <origin rpy="0.0 0.0 0.0" xyz="0.0 0.0 0.0"/>
+    </link>
+    <!-- attach extruder to tool0 -->
     <joint name="${prefix}extruder_attach_joint" type="fixed">
-      <parent link="${prefix}link_6"/>
-      <child link="${prefix}typhoon_extruder"/>
+      <parent link="${prefix}tool0"/>
+      <child link="${prefix}typhoon_extruder_base"/>
       <axis xyz="0 0 0"/>
       <origin rpy="0.0 0.0 0.0" xyz="0 0 0"/>
     </joint>
+    <joint name="${prefix}extruder_extruder_base" type="fixed">
+      <parent link="${prefix}typhoon_extruder_base"/>
+      <child link="${prefix}typhoon_extruder"/>
+      <axis xyz="0 0 0"/>
+      <origin rpy="0.0 0.0 0.0" xyz="0.159 0.0 0.08613"/>
+    </joint>
   </xacro:macro>
 </robot>
